Commit message: add udpate

File: boxbot_description/urdf/box_bot3.gazebo.xacro (robot description, xacro)
@@ -19,5 +19,5 @@
             <plugin name="camera_controller" filename="libgazebo_ros_camera.so">
                 <ros>
-                    <!-- <namespace>camera</namespace> -->
+                    <namespace>camera</namespace>
                     <remapping>camera/image_raw:=color/image_raw</remapping>
                     <remapping>camera/depth/image_raw:=depth/image_rect_raw</remapping>
@@ -41,5 +41,4 @@
             <joint_name>left_wheel_joint</joint_name>
             <joint_name>right_wheel_joint</joint_name>
-            <joint_name>laser_scan_link_joint</joint_name>
         </plugin>
     </gazebo>

File: boxbot_description/urdf/box_bot3.urdf.xacro (robot description, xacro)
@@ -22,5 +22,5 @@
         <visual>
             <geometry>
-                <mesh filename="package://my_box_bot_description/meshes/cute_cube.dae" scale="0.1 0.1 0.1"/>
+                <mesh filename="package://boxbot_description/meshes/cute_cube.dae" scale="0.1 0.1 0.1"/>
             </geometry>
         </visual>
@@ -116,5 +116,5 @@
             <origin xyz="0 0 0" rpy="0 0 0" />
             <geometry>
-                <mesh filename="package://my_box_bot_description/meshes/sensors/rplidar.dae" scale="1.0 1.0 1.0"/>
+                <mesh filename="package://boxbot_description/meshes/sensors/rplidar.dae" scale="1.0 1.0 1.0"/>
             </geometry>
         </visual>
