Commit message: add gazebo world

File: boxbot_description/urdf/box_bot3.urdf (robot description, URDF)
Before this commit: robot boxbot, 9 links, 8 joints
Links:
- added link camera_depth_optical_frame
Joints:
- added joint camera_optical_joint: type fixed, parent camera_link, child camera_depth_optical_frame, origin xyz=0 0 0 rpy=-1.57079632679 0 -1.57079632679
